File: frontgateschematic/frontgateschematic.sch (KiCad schematic (older format))
At the start: 9 parts

Commit message: Migrating to NodeMCU only
Parts:
- removed U? (x2): KQ330F, symbol jaidan:KQ330F
Changed lines of the file:
@@
 $EndDescr
-$Comp
-L jaidan:KQ330F U?
-U 1 1 6012A32B
-P 2000 3000
-F 0 "U?" H 4078 3451 50  0000 L CNN
-F 1 "KQ330F" H 4078 3360 50  0000 L CNN
-F 2 "" H 2000 3000 50  0001 C CNN
-F 3 "" H 2000 3000 50  0001 C CNN
-	1    2000 3000
-	1    0    0    -1
-$EndComp
-$Comp
-L jaidan:KQ330F U?
-U 1 1 6012AC75
-P 2000 9500
-F 0 "U?" H 4078 9951 50  0000 L CNN
-F 1 "KQ330F" H 4078 9860 50  0000 L CNN
-F 2 "" H 2000 9500 50  0001 C CNN
-F 3 "" H 2000 9500 50  0001 C CNN
-	1    2000 9500
-	1    0    0    -1
-$EndComp
 $Comp
 L arduino:Arduino_Mega2560_Shield XA?
@@
 	9000 1750 9100 1850
 Entry Wire Line
-	4650 4900 4750 5000
+	4650 5200 4750 5300
 Entry Wire Line
 	4650 5550 4750 5650
@@
 	5100 5650 4750 5650
 Wire Wire Line
-	5100 5050 4750 5050
-Wire Wire Line
-	4750 5050 4750 5000
+	5100 5350 4750 5350
+Wire Wire Line
+	4750 5350 4750 5300
 Wire Wire Line
 	9100 1850 9350 1850
@@
 Entry Wire Line
 	4850 1950 4950 1850
-Entry Wire Line
-	3650 3650 3750 3750
-Entry Wire Line
-	3750 3650 3850 3750
-Wire Wire Line
-	3750 3100 3750 3650
-Wire Wire Line
-	3650 3100 3650 3650
-Wire Bus Line
-	4550 4000 3600 4000
-Wire Bus Line
-	3600 4000 3600 3500
-Entry Wire Line
-	3500 3400 3600 3500
-Entry Wire Line
-	3400 3400 3500 3500
-Entry Wire Line
-	3300 3400 3400 3500
-Connection ~ 3600 4000
-Wire Bus Line
-	3600 4000 3500 4000
-Wire Wire Line
-	3500 3400 3500 3100
-Wire Wire Line
-	3500 3100 3550 3100
-Wire Wire Line
-	3400 3400 3400 3100
-Wire Wire Line
-	3400 3100 3450 3100
-Wire Wire Line
-	3300 3400 3300 3100
-Wire Wire Line
-	3300 3100 3350 3100
-Entry Bus Bus
-	4550 4000 4650 4100
 Wire Wire Line
 	4950 1850 5100 1850
@@
 	8700 2400 9350 2400
 Wire Bus Line
+	8000 4600 8600 4600
+Entry Wire Line
+	7050 10350 7150 10250
+Entry Wire Line
+	9950 9650 10050 9750
+Entry Wire Line
+	9950 9550 10050 9650
+Wire Wire Line
+	9950 9550 9400 9550
+Wire Wire Line
+	9950 9650 9400 9650
+Wire Bus Line
+	4850 3750 4400 3750
+Entry Wire Line
+	4400 4950 4500 5050
+Wire Wire Line
+	4500 5050 5100 5050
+Wire Bus Line
 	4650 6800 9000 6800
-Wire Bus Line
-	8000 3000 8600 3000
-Wire Bus Line
-	3750 3750 4850 3750
+Wire Wire Line
+	7800 9450 7150 9450
+Wire Wire Line
+	7150 9450 7150 10250
+Entry Wire Line
+	7700 2850 7800 2750
+Entry Wire Line
+	7700 2950 7800 2850
+Entry Wire Line
+	7700 3050 7800 2950
+Entry Wire Line
+	7700 3150 7800 3050
+Entry Wire Line
+	7700 1650 7800 1550
+Entry Wire Line
+	5000 1550 5100 1650
+Entry Wire Line
+	5000 2850 5100 2950
+Wire Bus Line
+	4400 3750 4400 10350
+Wire Bus Line
+	10050 9650 10050 10350
+Wire Bus Line
+	4400 10350 10050 10350
+Wire Bus Line
+	4650 5200 4650 6800
 Wire Bus Line
 	9000 1750 9000 6800
 Wire Bus Line
-	4650 4100 4650 6800
-Wire Bus Line
 	4850 1750 4850 3750
 Wire Bus Line
-	3350 3500 3600 3500
-Wire Bus Line
-	8000 3000 8000 5100
-Wire Bus Line
-	8600 2000 8600 3000
+	8000 4600 8000 5100
+Wire Bus Line
+	8600 2000 8600 4600
 $EndSCHEMATC
